File: hardware/midi-switcher.sch (EAGLE design)
At the start: 70 parts, among them IC1 PIC16F1825DIL14, IC2 6N138

Commit message: fix eagle consistency error
Parts:
- R10, R11, R12, R13, R14, R15, R16, R17, R18, R19, R20, R21, R6, R7, R8, R9: device rcl:R-EU_0207/2V -> rcl:R-EU_0207/7
Changed lines of the file:
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@@
 <?xml version="1.0" encoding="utf-8"?>
 <!DOCTYPE eagle SYSTEM "eagle.dtd">
-<eagle version="6.4">
+<eagle version="6.6.0">
 <drawing>
 <settings>
@@
 <part name="R3" library="rcl" deviceset="R-EU_" device="0207/7"/>
 <part name="C2" library="rcl" deviceset="C-EU" device="025-025X050"/>
-<part name="R15" library="rcl" deviceset="R-EU_" device="0207/2V"/>
-<part name="R17" library="rcl" deviceset="R-EU_" device="0207/2V"/>
-<part name="R19" library="rcl" deviceset="R-EU_" device="0207/2V"/>
-<part name="R21" library="rcl" deviceset="R-EU_" device="0207/2V"/>
-<part name="R13" library="rcl" deviceset="R-EU_" device="0207/2V"/>
-<part name="R11" library="rcl" deviceset="R-EU_" device="0207/2V"/>
-<part name="R9" library="rcl" deviceset="R-EU_" device="0207/2V"/>
-<part name="R7" library="rcl" deviceset="R-EU_" device="0207/2V"/>
+<part name="R15" library="rcl" deviceset="R-EU_" device="0207/7"/>
+<part name="R17" library="rcl" deviceset="R-EU_" device="0207/7"/>
+<part name="R19" library="rcl" deviceset="R-EU_" device="0207/7"/>
+<part name="R21" library="rcl" deviceset="R-EU_" device="0207/7"/>
+<part name="R13" library="rcl" deviceset="R-EU_" device="0207/7"/>
+<part name="R11" library="rcl" deviceset="R-EU_" device="0207/7"/>
+<part name="R9" library="rcl" deviceset="R-EU_" device="0207/7"/>
+<part name="R7" library="rcl" deviceset="R-EU_" device="0207/7"/>
 <part name="ICSP" library="microbuilder" deviceset="HEADER-1X6" device=""/>
 <part name="OP1-" library="adafruit" deviceset="PINHD-1X1" device=""/>
@@
 <part name="C5" library="rcl" deviceset="CPOL-EU" device="E2.5-7"/>
 <part name="LED5" library="adafruit" deviceset="LED" device="3MM"/>
-<part name="R14" library="rcl" deviceset="R-EU_" device="0207/2V"/>
-<part name="R16" library="rcl" deviceset="R-EU_" device="0207/2V"/>
-<part name="R18" library="rcl" deviceset="R-EU_" device="0207/2V"/>
-<part name="R20" library="rcl" deviceset="R-EU_" device="0207/2V"/>
-<part name="R12" library="rcl" deviceset="R-EU_" device="0207/2V"/>
-<part name="R10" library="rcl" deviceset="R-EU_" device="0207/2V"/>
-<part name="R8" library="rcl" deviceset="R-EU_" device="0207/2V"/>
-<part name="R6" library="rcl" deviceset="R-EU_" device="0207/2V"/>
+<part name="R14" library="rcl" deviceset="R-EU_" device="0207/7"/>
+<part name="R16" library="rcl" deviceset="R-EU_" device="0207/7"/>
+<part name="R18" library="rcl" deviceset="R-EU_" device="0207/7"/>
+<part name="R20" library="rcl" deviceset="R-EU_" device="0207/7"/>
+<part name="R12" library="rcl" deviceset="R-EU_" device="0207/7"/>
+<part name="R10" library="rcl" deviceset="R-EU_" device="0207/7"/>
+<part name="R8" library="rcl" deviceset="R-EU_" device="0207/7"/>
+<part name="R6" library="rcl" deviceset="R-EU_" device="0207/7"/>
 <part name="LED_6" library="adafruit" deviceset="LED" device="3MM"/>
 <part name="LED_7" library="adafruit" deviceset="LED" device="3MM"/>
