File: smt-board/midi-switcher-smt.sch (EAGLE design)
At the start: 70 parts, among them IC1 PIC16F1825DIL14, IC2 6N138, Q1 MJD122GDPAK, Q2 MJD122GDPAK, Q3 MJD122GDPAK, Q4 MJD122GDPAK, Q5 MJD122GDPAK, Q6 MJD122GDPAK, Q7 MJD122GDPAK, Q8 MJD122GDPAK

Commit message: version 7
Parts:
- D1: device adafruit:DIODE_SOD-123FL -> adafruit:DIODESMA
Changed lines of the file:
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@@
 <part name="Q8" library="jason_eagle6" deviceset="MJD122G" device="DPAK"/>
 <part name="D2" library="jasons_stuff" deviceset="0805DIODE" device=""/>
-<part name="D1" library="adafruit" deviceset="DIODE" device="_SOD-123FL"/>
+<part name="D1" library="adafruit" deviceset="DIODE" device="SMA"/>
 <part name="REG1" library="jason_eagle6" deviceset="LD1086" device=""/>
 </parts>

Commit message: new layout
Parts:
- removed JP18, JP19: (no value), adafruit:PINHD-1X1
- added D3: 1N4004, jasons_stuff:1N4004
- added JP1, JP2, POWER+1, POWER+2, POWER-1, POWER-2: (no value), adafruit:PINHD-1X1
- added JP3: (no value), pinhead:PINHD-1X3
- added R22: (no value), rcl:R-EU_R0805
- added T1: (no value), transistor:MMBT3906LT1-PNP-SOT23-BEC
- added U$1: 2.1MMJACKTHM, adafruit:2.1MMJACKTHM
- C4: device rcl:CPOL-EUF -> rcl:CPOL-EUE2.5-7
- C5: device rcl:CPOL-EUD -> rcl:CPOL-EUE2.5-6
- D1: value (none) -> 1N4004; device adafruit:DIODESMA -> jasons_stuff:1N4004
- IC1: value PIC16F1825DIL14 -> PIC16F1825SO14; device jasons_stuff:PIC16F1825DIL14 -> jasons_stuff:PIC16F1825SO14
Connections:
- removed net N$44: IC1.RA4/SDO, MODE.S, MODE.S1
- new net N$32: IC1.RA3/MCLR#/VPP, ICSP.1, MODE.P, MODE.P1
- new net N$40: JP1.1, R22.2
- new net N$41: D1.A, D3.C, JP3.2
- new net N$43: D3.A, U$1.TIP
- net 12V: now also JP3.3, POWER+1.1, POWER+2.1; no longer D1.A, JP18.1
- net GND: now also MODE.S, MODE.S1, POWER-1.1, POWER-2.1, T1.C, U$1.RING; no longer JP19.1, MODE.P, MODE.P1
- net N$16: now also JP2.1, T1.E
- net N$23: now also IC1.RA4/SDO; no longer IC1.RC4/TX
- net N$34: now also R22.1, T1.B; no longer IC1.RA3/MCLR#/VPP, ICSP.1
Other:
- moved on the sheet: C4, C5, MODE, R4

Commit message: updates
Parts:
- removed 12V, JP1, JP2: (no value), adafruit:PINHD-1X1
- removed ACT, LED1, LED2, LED3, LED4, LED5, LED8, LED_6, LED_7, PWR: (no value), led:LEDCHIP-LED0805
- removed R4, R5, R6: (no value), rcl:R-EU_R0805
- removed REG1: LD1086, jason_eagle6:LD1086
- removed T1: (no value), transistor:MMBT3906LT1-PNP-SOT23-BEC
- added CHAIN_NEXT, CHAIN_PREV, OP8+1: (no value), adafruit:PINHD-1X1
- added IC3: LD1086, jason_eagle6:LD1086
- added L1, L10, L2, L3, L4, L5, L6, L7, L8, L9: (no value), led:LEDCHIP-LED0805
- added Q9: (no value), transistor:MMBT3906LT1-PNP-SOT23-BEC
- added R23, R24, R25: (no value), rcl:R-EU_R0805
- D1: value 1N4004 -> 0805DIODE; device jasons_stuff:1N4004 -> jasons_stuff:0805DIODE
- D2: value 0805DIODE -> 1N4004; device jasons_stuff:0805DIODE -> jasons_stuff:1N4004
- IC1: value PIC16F1825SO14 -> 6N138; device jasons_stuff:PIC16F1825SO14 -> optocoupler:6N138
- IC2: value 6N138 -> PIC16F1825SO14; device optocoupler:6N138 -> jasons_stuff:PIC16F1825SO14
Connections:
- removed net 12V: 12V.1, JP3.3, OP1+.1, OP2+.1, OP3+.1, OP4+.1, OP5+.1, OP7+.1, OP8+.1, POWER+1.1, POWER+2.1
- removed net N$11 (its old number): Q4.B, R21.1
- removed net N$17: IC1.RA5, R4.1
- removed net N$19: IC1.RA0/ICSPDAT, ICSP.4, R20.1, R21.2
- removed net N$2 (its old number): D2.P$2, IC2.A, R1.1
- removed net N$20: IC1.RC2, R12.1, R13.2
- removed net N$21: IC1.RC3/SS#, R10.1, R11.2
- removed net N$22: IC1.RC1/SDA/SDI, R8.1, R9.2
- removed net N$23: IC1.RA4/SDO, R6.1, R7.2
- removed net N$32: IC1.RA3/MCLR#/VPP, ICSP.1, MODE.P, MODE.P1
- removed net N$34: R22.1, T1.B
- removed net N$40: JP1.1, R22.2
- removed net N$41: D1.A, D3.C, JP3.2
- removed net N$45: IC1.RA2/INT, R16.1, R17.2
- removed net N$46: IC1.RCO/SCL/SCK, R14.1, R15.2
- removed net VDD: C2.1, C3.2, C5.+, IC1.VDD, IC2.VCC, ICSP.2, R3.1, R5.2, REG1.OUT
- new net +12V: JP3.2, JP3.3, OP1+.1, OP2+.1, OP3+.1, OP4+.1, OP5+.1, OP7+.1, OP8+.1, OP8+1.1, POWER+1.1, POWER+2.1
- new net +5V: C1.2, C2.1, C5.+, IC1.VCC, IC2.VDD, IC3.OUT, ICSP.2, L2.A, R22.2
- new net ACT_LED: IC2.RA4/SDO, L1.A
- new net MIDI_IN: CHAIN_NEXT.1, IC1.VO, IC2.RA1/ICPCLK, ICSP.5, Q9.E, R22.1
- new net N$1: D1.P$1, IC1.C, MIDI_IN.5
- new net N$12: Q4.B, R11.1
- new net N$51: IC2.RA0/ICSPDAT, ICSP.4
- new net N$54: D2.C, D3.A, JP3.1
- new net OUT1: IC2.RA5, R19.2, R20.1
- new net OUT2: IC2.RC5/RX, R17.2, R18.1
- new net OUT3: IC2.RC1/SDA/SDI, R15.2, R16.1
- new net OUT4: IC2.RA2/INT, R13.2, R14.1
- new net OUT5: IC2.RC4/TX, R11.2, R12.1
- new net OUT6: IC2.RC3/SS#, R10.1, R9.2
- new net OUT7: IC2.RC2, R7.2, R8.1
- new net OUT8: IC2.RCO/SCL/SCK, R2.2, R3.1
- new net SWITCH: IC2.RA3/MCLR#/VPP, ICSP.1, MODE.S, MODE.S1
- net GND: now also IC1.GND, IC2.VSS, IC3.GND, L10.C, L3.C, L4.C, L5.C, L6.C, L7.C, L8.C, L9.C, MODE.P, MODE.P1, Q9.C, R21.1, R24.2, R25.2; no longer ACT.C, IC1.VSS, IC2.GND, LED1.C, LED2.C, LED3.C, LED4.C, LED5.C, LED8.C, LED_6.C, LED_7.C, MODE.S, MODE.S1, PWR.C, R2.1, REG1.GND, T1.C
- net N$10: now also Q6.B, R15.1; no longer Q3.B, R19.1
- net N$13: now also Q3.B, R9.1; no longer Q6.B, R11.1
- net N$14: now also Q2.B, R7.1; no longer Q7.B, R9.1
- net N$15: now also Q1.B, R2.1; no longer Q8.B, R7.1
- net N$16: now also Q9.B, R23.2; no longer IC1.RC5/RX, IC2.VO, JP2.1, R3.2, T1.E
- net N$18: now also CHAIN_PREV.1, R23.1; no longer IC1.RA1/ICPCLK, ICSP.5, R18.1, R19.2
- net N$24: now also L8.A, R16.2; no longer LED_7.A, R18.2
- net N$25: now also Q8.C; no longer Q1.C
- net N$26: now also Q7.C; no longer Q2.C
- net N$27: now also Q6.C; no longer Q3.C
- net N$28: now also L2.C, R24.1; no longer PWR.A, R5.1
- net N$29: now also Q4.C; no longer Q5.C
- net N$3: now also D1.P$2, IC1.A, R1.1; no longer D2.P$1, IC2.C, MIDI_IN.5
- net N$30: now also Q3.C; no longer Q6.C
- net N$31: now also Q5.C; no longer Q4.C
- net N$33: now also L7.A, R14.2; no longer LED8.A, R20.2
- net N$35: now also L6.A; no longer LED4.A
- net N$36: now also L5.A; no longer LED3.A
- net N$37: now also L4.A; no longer LED2.A
- net N$38: now also L3.A, R3.2; no longer LED1.A, R6.2
- net N$39: now also C3.2, D3.C, IC3.IN; no longer C1.2, D1.C, REG1.IN
- net N$4: now also IC1.VB, R21.2; no longer IC2.VB, R2.2
- net N$42: now also Q2.C; no longer Q7.C
- net N$43: now also D2.A; no longer D3.A
- net N$47: now also Q1.C; no longer Q8.C
- net N$5: now also L1.C, R25.1; no longer ACT.A, R4.2
- net N$6: now also L10.A, R20.2; no longer LED5.A, R14.2
- net N$7: now also L9.A, R18.2; no longer LED_6.A, R16.2
- net N$8: now also Q8.B, R19.1; no longer Q1.B, R15.1
- net N$9: now also Q7.B; no longer Q2.B
Other:
- note added: "MICROCONTROLLER PIC16F1825"
- note added: "MIDI INPUT CIRCUIT"
- note added: "MIDI SWITCHER"
- note added: "OUTPUT DRIVERS"
- note added: "OUTPUT STATE LEDS"
- note added: "POWER SUPPLY"
- note added: "SMT layout. Version 7, July 2017 Jason Hotchkiss, Sixty Four Pixels Ltd"
- note added: "{ FAST { PWM { CAPABLE { {"
- moved on the sheet: C1, C3, C4, C5, D3, JP3, MIDI_IN, MODE, OP1+, OP1-, OP2+, OP2-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
