File: smt-board/midi-switcher-smt.brd (EAGLE design)
At the start: 104.1 x 35.6 mm, 79 parts, among them IC1 6N138, IC2 PIC16F1825SO14, IC3 LD1086, Q1 MJD122GDPAK, Q2 MJD122GDPAK, Q3 MJD122GDPAK, Q4 MJD122GDPAK, Q5 MJD122GDPAK, Q6 MJD122GDPAK, Q7 MJD122GDPAK, Q8 MJD122GDPAK

Commit message: done?
Other:
- board size 104.1 x 35.6 mm -> 104.1 x 38.1 mm
- board text added: "++"
- board text added: "--A"
- board text added: "--B"
- board text added: "--C"
- board text added: "--D"
- board text added: "--E"
- board text added: "--F"
- board text added: "--G"
- board text added: "--H"
- board text added: "GROUND"
- board text added: "POWER IN"
- board text removed: "+"
- board text removed: "-"
- board text removed: "Outputs"
Changed lines of the file:
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@@
 <rectangle x1="85.40115" y1="19.65325" x2="85.47735" y2="19.69135" layer="52" rot="R180"/>
 <rectangle x1="88.98255" y1="19.69135" x2="89.02065" y2="19.72945" layer="52" rot="R180"/>
-<wire x1="13.97" y1="5.08" x2="115.57" y2="5.08" width="0.4064" layer="20"/>
-<wire x1="116.84" y1="6.35" x2="116.84" y2="39.37" width="0.4064" layer="20"/>
+<wire x1="13.97" y1="2.54" x2="115.57" y2="2.54" width="0.4064" layer="20"/>
+<wire x1="116.84" y1="3.81" x2="116.84" y2="39.37" width="0.4064" layer="20"/>
 <wire x1="115.57" y1="40.64" x2="13.97" y2="40.64" width="0.4064" layer="20"/>
-<hole x="16.51" y="15.24" drill="3.2"/>
-<hole x="113.03" y="15.24" drill="3.2"/>
+<hole x="16.51" y="13.97" drill="3.2"/>
+<hole x="113.03" y="13.97" drill="3.2"/>
 <hole x="69.85" y="38.1" drill="3.2"/>
 <text x="28.321" y="15.494" size="2.54" layer="51" font="vector">A</text>
@@
 <text x="79.121" y="15.494" size="2.54" layer="51" font="vector">F</text>
 <text x="89.281" y="15.494" size="2.54" layer="51" font="vector">G</text>
-<text x="18.161" y="10.922" size="2.54" layer="51" font="vector">+</text>
-<text x="109.601" y="10.795" size="2.54" layer="51" font="vector">-</text>
-<circle x="19.05" y="12.192" radius="1.27" width="0.3048" layer="51"/>
-<circle x="110.49" y="12.065" radius="1.27" width="0.3048" layer="51"/>
-<wire x1="12.7" y1="39.37" x2="12.7" y2="6.35" width="0.4064" layer="20"/>
+<wire x1="12.7" y1="39.37" x2="12.7" y2="3.81" width="0.4064" layer="20"/>
 <wire x1="115.57" y1="40.64" x2="116.84" y2="39.37" width="0.3048" layer="20" curve="-90"/>
-<wire x1="116.84" y1="6.35" x2="115.57" y2="5.08" width="0.3048" layer="20" curve="-90"/>
-<wire x1="13.97" y1="5.08" x2="12.7" y2="6.35" width="0.3048" layer="20" curve="-90"/>
+<wire x1="116.84" y1="3.81" x2="115.57" y2="2.54" width="0.3048" layer="20" curve="-90"/>
+<wire x1="13.97" y1="2.54" x2="12.7" y2="3.81" width="0.3048" layer="20" curve="-90"/>
 <wire x1="12.7" y1="39.37" x2="13.97" y2="40.64" width="0.3048" layer="20" curve="-90"/>
 <wire x1="44.958" y1="39.37" x2="44.958" y2="36.83" width="0.3048" layer="51"/>
@@
   R20</text>
 <wire x1="27.686" y1="23.495" x2="33.147" y2="23.495" width="0.254" layer="21"/>
-<wire x1="13.589" y1="23.749" x2="13.589" y2="19.939" width="0.3048" layer="21"/>
-<wire x1="13.589" y1="19.939" x2="19.939" y2="19.939" width="0.3048" layer="21"/>
-<wire x1="19.939" y1="19.939" x2="19.939" y2="23.749" width="0.3048" layer="21"/>
-<wire x1="19.939" y1="23.749" x2="13.589" y2="23.749" width="0.3048" layer="21"/>
-<circle x="15.24" y="21.844" radius="0.851940625" width="0.3048" layer="21"/>
-<circle x="18.288" y="21.844" radius="0.851940625" width="0.3048" layer="21"/>
-<wire x1="18.288" y1="22.606" x2="18.288" y2="21.082" width="0.3048" layer="21"/>
-<wire x1="17.526" y1="21.844" x2="19.05" y2="21.844" width="0.3048" layer="21"/>
-<wire x1="14.478" y1="21.844" x2="16.002" y2="21.844" width="0.3048" layer="21"/>
 <text x="28.321" y="12.065" size="2.54" layer="51" font="vector">~</text>
 <text x="38.481" y="12.065" size="2.54" layer="51" font="vector">~</text>
 <text x="48.641" y="12.065" size="2.54" layer="51" font="vector">~</text>
 <text x="58.801" y="12.065" size="2.54" layer="51" font="vector">~</text>
-<text x="13.335" y="18.288" size="1.27" layer="25" font="vector">Outputs</text>
 <circle x="49.022" y="39.497" radius="0.523634375" width="0.3048" layer="21"/>
 <text x="66.294" y="35.814" size="1.27" layer="25" font="vector" rot="R90">ICSP</text>
@@
 <text x="49.53" y="13.97" size="1.778" layer="22" font="vector" rot="MR0">six4pix.com/switcher</text>
 <text x="99.441" y="15.494" size="2.54" layer="51" font="vector">H</text>
-<wire x1="14.5" y1="10" x2="14.5" y2="6" width="0.4064" layer="21"/>
+<wire x1="14.5" y1="10" x2="14.5" y2="2.698" width="0.4064" layer="21"/>
 <wire x1="14.5" y1="10" x2="24.5" y2="10" width="0.4064" layer="21"/>
 <wire x1="24.5" y1="10" x2="34.5" y2="10" width="0.4064" layer="21"/>
@@
 <wire x1="94.5" y1="10" x2="104.5" y2="10" width="0.4064" layer="21"/>
 <wire x1="104.5" y1="10" x2="114.5" y2="10" width="0.4064" layer="21"/>
-<wire x1="114.5" y1="10" x2="114.5" y2="6" width="0.4064" layer="21"/>
-<wire x1="104.5" y1="10" x2="104.5" y2="6" width="0.4064" layer="21"/>
-<wire x1="94.5" y1="10" x2="94.5" y2="6" width="0.4064" layer="21"/>
-<wire x1="84.5" y1="10" x2="84.5" y2="6" width="0.4064" layer="21"/>
-<wire x1="74.5" y1="10" x2="74.5" y2="6" width="0.4064" layer="21"/>
-<wire x1="64.5" y1="10" x2="64.5" y2="6" width="0.4064" layer="21"/>
-<wire x1="54.5" y1="10" x2="54.5" y2="6" width="0.4064" layer="21"/>
-<wire x1="44.5" y1="10" x2="44.5" y2="6" width="0.4064" layer="21"/>
-<wire x1="34.5" y1="10" x2="34.5" y2="6" width="0.4064" layer="21"/>
-<wire x1="24.5" y1="10" x2="24.5" y2="6" width="0.4064" layer="21"/>
-<rectangle x1="104.267" y1="5.588" x2="114.681" y2="10.033" layer="21"/>
-<rectangle x1="14.351" y1="5.588" x2="24.638" y2="10.033" layer="21"/>
+<wire x1="114.5" y1="10" x2="114.5" y2="2.698" width="0.4064" layer="21"/>
+<wire x1="104.5" y1="10" x2="104.5" y2="2.698" width="0.4064" layer="21"/>
+<wire x1="94.5" y1="10" x2="94.5" y2="2.698" width="0.4064" layer="21"/>
+<wire x1="84.5" y1="10" x2="84.5" y2="2.698" width="0.4064" layer="21"/>
+<wire x1="74.5" y1="10" x2="74.5" y2="2.698" width="0.4064" layer="21"/>
+<wire x1="64.5" y1="10" x2="64.5" y2="2.698" width="0.4064" layer="21"/>
+<wire x1="54.5" y1="10" x2="54.5" y2="2.698" width="0.4064" layer="21"/>
+<wire x1="44.5" y1="10" x2="44.5" y2="2.571" width="0.4064" layer="21"/>
+<wire x1="34.5" y1="10" x2="34.5" y2="2.698" width="0.4064" layer="21"/>
+<wire x1="24.5" y1="10" x2="24.5" y2="2.698" width="0.4064" layer="21"/>
+<wire x1="29.21" y1="10.033" x2="29.21" y2="13.843" width="0.3048" layer="21"/>
+<wire x1="39.37" y1="10.033" x2="39.37" y2="13.843" width="0.3048" layer="21"/>
+<wire x1="49.53" y1="10.033" x2="49.53" y2="13.843" width="0.3048" layer="21"/>
+<wire x1="59.69" y1="10.033" x2="59.69" y2="13.843" width="0.3048" layer="21"/>
+<wire x1="69.85" y1="10.033" x2="69.85" y2="13.843" width="0.3048" layer="21"/>
+<wire x1="80.01" y1="10.033" x2="80.01" y2="13.843" width="0.3048" layer="21"/>
+<wire x1="90.17" y1="10.033" x2="90.17" y2="13.843" width="0.3048" layer="21"/>
+<text x="33.02" y="3.175" size="1.27" layer="21" font="vector" rot="MR0">++</text>
+<text x="42.926" y="3.175" size="1.27" layer="21" font="vector" rot="MR0">++</text>
+<text x="52.959" y="3.175" size="1.27" layer="21" font="vector" rot="MR0">++</text>
+<text x="62.865" y="3.175" size="1.27" layer="21" font="vector" rot="MR0">++</text>
+<text x="73.152" y="3.175" size="1.27" layer="21" font="vector" rot="MR0">++</text>
+<text x="82.931" y="3.175" size="1.27" layer="21" font="vector" rot="MR0">++</text>
+<text x="92.964" y="3.175" size="1.27" layer="21" font="vector" rot="MR0">++</text>
+<text x="102.997" y="3.175" size="1.27" layer="21" font="vector" rot="MR0">++</text>
+<text x="25.4" y="3.175" size="1.27" layer="21" font="vector">--A</text>
+<text x="35.56" y="3.175" size="1.27" layer="21" font="vector">--B</text>
+<text x="45.339" y="3.175" size="1.27" layer="21" font="vector">--C</text>
+<text x="55.499" y="3.175" size="1.27" layer="21" font="vector">--D</text>
+<text x="65.405" y="3.175" size="1.27" layer="21" font="vector">--E</text>
+<text x="75.438" y="3.175" size="1.27" layer="21" font="vector">--F</text>
+<text x="85.344" y="3.175" size="1.27" layer="21" font="vector">--G</text>
+<text x="95.377" y="3.175" size="1.27" layer="21" font="vector">--H</text>
+<text x="14.986" y="3.175" size="1.27" layer="21" font="vector">POWER IN</text>
+<text x="106.172" y="3.175" size="1.27" layer="21" font="vector">GROUND</text>
 </plain>
 <attributes>
@@
 </element>
 <element name="C3" library="rcl" package="C0805" value="" x="106.68" y="24.13" smashed="yes" rot="R180">
-<attribute name="NAME" x="106.553" y="26.543" size="1.27" layer="25" ratio="10" rot="R180"/>
+<attribute name="NAME" x="106.426" y="26.67" size="1.27" layer="25" ratio="10" rot="R180"/>
 <attribute name="VALUE" x="108.966" y="26.924" size="1.27" layer="27" ratio="10" rot="R180"/>
 </element>
@@
 </element>
 <element name="C4" library="rcl" package="E2,5-7" value="" x="99.441" y="29.464" smashed="yes" rot="R180">
-<attribute name="NAME" x="103.886" y="26.797" size="1.27" layer="25" ratio="10" rot="R180"/>
+<attribute name="NAME" x="104.013" y="33.147" size="1.27" layer="25" ratio="10" rot="R180"/>
 <attribute name="VALUE" x="96.393" y="32.639" size="1.27" layer="27" ratio="10" rot="R180"/>
 </element>
