File: smt-relay-module/midi-switcher-smt-relay.brd (EAGLE design)
At the start: 105.5 x 47.7 mm, 100 parts, among them IC1 6N138, IC2 PIC16F1825SO14, IC3 SP34063A_BOOST_REG

Commit message: REED RELAY MODULE REV1
Parts:
- renumbered RLY1 to RL1, RLY2 to RL3, RLY3 to RL5, RLY4 to RL7, RLY5 to RL2, RLY6 to RL4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
Other:
- board text added: "R13 .. R25"
