File: smt-relay-module/midi-switcher-smt-relay.sch (EAGLE design)
At the start: 100 parts, among them IC1 6N138, IC2 PIC16F1825SO14, IC3 SP34063A_BOOST_REG

Commit message: REED RELAY MODULE REV1
Parts:
- renumbered RLY1 to RL1, RLY2 to RL3, RLY3 to RL5, RLY4 to RL7, RLY5 to RL2, RLY6 to RL4, RLY7 to RL6, RLY8 to RL8
Other:
- note added: "MIDI BUS"
- note added: "MIDI SWITCHER: REED RELAYS OUTPUTS"
- note added: "POWER INPUT"
- note added: "REED RELAYS"
- note added: "REV 1, 30 JAN 2018. Jason Hotchkiss / Sixty Four Pixels Ltd"
- moved on the sheet: C2, C3, C4, C5, D10, D11, D12, D13, D14, L1, L2, LED1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
