File: midi_switcher_trs/midi_switcher_trs.brd (EAGLE design)
At the start: 152.4 x 43.4 mm, 83 parts, among them IC1 PIC16F1825SO14, IC2 REG1117, IC3 6N138, IC4 MB1S, X1 ACJM-MHDRA, X2 ACJM-MHDRA, X3 ACJM-MHDRA, X4 ACJM-MHDRA, X6 VERTICAL_3_5MM_SOCKET

Commit message: V2
Parts:
- removed IC4: MB1S, rectifier:SOIC-4
- removed L3, L4, L5, L6, L7, L8: (no value), led:LED3MM
- removed RR7, RR8: (no value), rcl:R0805
- added A, B, C, D, E, F, G, H: (no value), led:LED3MM
- added D11, D12: 0805DIODE, jasons_stuff:0805DIODE
- added R22, R23, R24, R7, R8: (no value), rcl:R0805
- C3: device rcl:C0805 -> rcl:E2,5-7
- C4, C5: device rcl:E2,5-6E -> rcl:E2,5-7
- D1: value CGRM4001-G -> (none); device diode:SOD-123_MINI-SMA -> microbuilder:SOD-123
- D2: value 0805DIODE -> CGRM4001-G; device jasons_stuff:0805DIODE -> diode:SOD-123_MINI-SMA
- D3: value 0805DIODE -> (none); device jasons_stuff:0805DIODE -> microbuilder:SOD-123
- IC1: value PIC16F1825SO14 -> SP34063A_BOOST_REG; device jasons_stuff:SO14 -> jason_eagle6:SOIC8
- IC2: value REG1117 -> PIC16F1825SO14; device burr-brown:SOT223 -> jasons_stuff:SO14
- L1: device led:LED3MM -> SparkFun:1210
- L2: device led:LED3MM -> inductors:DR1030
- moved R15 108.1 mm to (21.6, 38.9), turned to 180 degrees
- moved R14 101.3 mm to (34.0, 37.8), turned to 270 degrees
- moved D4 98.1 mm to (25.1, 35.1), turned to 270 degrees
- moved D3 78.9 mm to (66.0, 40.6), turned to 180 degrees
- moved R16 75.9 mm to (31.0, 32.8), turned to 270 degrees
- moved D2 70.9 mm to (95.9, 30.9), turned to 180 degrees
- moved R13 64.9 mm to (86.4, 35.6), turned to 90 degrees
- moved R11 56.2 mm to (90.2, 40.6), turned to 180 degrees
- moved R12 54.5 mm to (85.1, 39.4), turned to 180 degrees
- moved R20 51.3 mm to (99.1, 14.5)
- moved R18 50.9 mm to (127.0, 14.7)
- moved D1 34.9 mm to (129.5, 31.8), turned to 180 degrees
- moved R21 33.1 mm to (76.2, 12.4)
- moved R17 33.1 mm to (132.1, 12.4)
- moved R19 33.1 mm to (104.1, 12.4)
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Connections:
- removed net N$43: C2.1, C4.+, IC2.3, IC4.+
- new net +9V: C5.+, D1.C, IC1.6, R11.1
- new net N$42: D1.A, U$9.BARREL
- new net N$44: IC1.1, IC1.7, IC1.8, R11.2
- new net N$45: C1.1, IC1.3
- new net N$57: C4.+, L1.1, L2.1, R12.1
- net BUTTON: now also IC2.2; no longer IC1.2
- net GND: now also C3.-, D2.A, IC1.4, IC2.14, R13.1, R14.1, R7.2, R8.2, U$9.PIN; no longer C3.2, IC1.14, IC2.1, IC4.-, R11.1, RR7.2, RR8.2
- net LED: now also IC2.3; no longer IC1.3
- net MIDI_IN: now also IC2.5, R16.2; no longer IC1.5, R12.2
- net N$10: now also D12.C; no longer D10.C
- net N$15: now also D10.C; no longer D8.C
- net N$16: now also D9.C; no longer D7.C
- net N$17: now also R22.1; no longer R19.1
- net N$18: now also R21.1; no longer R18.1
- net N$24: now also D8.C; no longer D6.C
- net N$25: now also D7.C; no longer D5.C
- net N$26: now also R20.1; no longer R17.1
- net N$27: now also R19.1; no longer R16.1
- net N$33: now also D6.C; no longer D4.C
- net N$34: now also D5.C; no longer D3.C
- net N$35: now also R18.1; no longer R15.1
- net N$36: now also R17.1; no longer R14.1
- net N$37: now also D4.C; no longer D2.C
- net N$38: now also R15.1; no longer R13.1
- net N$39: now also D4.A, R15.2; no longer D2.A, R13.2
- net N$40: now also R14.2; no longer R11.2
- net N$41: now also R1.1; no longer R3.1
- net N$46: now also D2.C, IC1.2, L2.2; no longer IC4.~1, U$9.BARREL
- net N$47: now also IC1.5, R12.2, R13.2; no longer IC4.~2, U$9.PIN
- net N$48: now also R2.1; no longer R4.1
- net N$49: now also A.K; no longer L1.K
- net N$50: now also B.K; no longer L2.K
- net N$51: now also C.K, R8.1; no longer L3.K, RR8.1
- net N$52: now also D.K, R7.1; no longer L4.K, RR7.1
- net N$53: now also E.K; no longer L5.K
- net N$54: now also F.K; no longer L6.K
- net N$55: now also G.K, R4.1; no longer L7.K, R2.1
- net N$56: now also H.K, R3.1; no longer L8.K, R1.1
- net N$6: now also D11.C; no longer D9.C
- net N$7: now also R24.1; no longer R21.1
- net N$8: now also R23.1; no longer R20.1
- net SUPPLY: now also C3.+, D11.A, D12.A, L1.2; no longer C1.1, C5.+, D1.A, D4.A, IC2.2
- net TRIG1: now also A.A, IC2.13, R24.2; no longer IC1.13, L1.A, R21.2
- net TRIG2: now also B.A, IC2.12, R23.2; no longer IC1.12, L2.A, R20.2
- net TRIG3: now also C.A, IC2.8, R22.2; no longer IC1.8, L3.A, R19.2
- net TRIG4: now also D.A, IC2.9, R21.2; no longer IC1.9, L4.A, R18.2
- net TRIG5: now also E.A, IC2.10, R20.2; no longer IC1.10, L5.A, R17.2
- net TRIG6: now also F.A, IC2.11, R19.2; no longer IC1.11, L6.A, R16.2
- net TRIG7: now also G.A, IC2.7, R18.2; no longer IC1.7, L7.A, R15.2
- net TRIG8: now also H.A, IC2.6, R17.2; no longer IC1.6, L8.A, R14.2
- net VDD: now also C2.1, D3.C, IC2.1, R16.1; no longer C3.1, D1.C, IC1.1, R12.1
- net VPP: now also IC2.4; no longer IC1.4
Routing:
- net SUPPLY: track 258.8 -> 195.6 mm
- net +9V: track 0.00 -> 46.6 mm, vias 0 -> 1
- net TRIG2: track 53.3 -> 96.9 mm, vias 0 -> 5
- net N$43: track 37.8 -> 0.00 mm
- net N$13: track 70.6 -> 38.4 mm
- net N$4: track 71.8 -> 39.7 mm
- net N$22: track 70.5 -> 38.7 mm
- net N$31: track 70.2 -> 39.7 mm
- net N$47: track 33.4 -> 4.92 mm, vias 1 -> 0
- net VDD: track 148.1 -> 127.3 mm, vias 5 -> 2
- net N$46: track 32.6 -> 12.0 mm
- net N$57: track 0.00 -> 17.2 mm
- net N$3: track 39.6 -> 55.1 mm
- net N$12: track 38.7 -> 51.0 mm
- net N$30: track 38.9 -> 49.5 mm
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Other:
- board text added: "MIDI SWITCHER TRS REV 2"
- board text added: "Sixty Four Pixels"
- board text added: "six4pix.com/switchertrs"
- board text removed: "MIDI SWITCHER"
- board text removed: "TRS"
- board text removed: "rev 1"
- board text removed: "six4pix.com/switcher"
