File: midi_switcher_trs/midi_switcher_trs.sch (EAGLE design)
At the start: 83 parts, among them IC1 PIC16F1825SO14, IC2 REG1117, IC3 6N138, IC4 MB1S, X1 ACJM-MHDRA, X2 ACJM-MHDRA, X3 ACJM-MHDRA, X4 ACJM-MHDRA, X6 VERTICAL_3_5MM_SOCKET

Commit message: V2
Parts:
- removed IC4: MB1S, rectifier:MB1S
- added A, B: (no value), led:LED3MM
- added D11, D12: 0805DIODE, jasons_stuff:0805DIODE
- added R22, R23, R24: (no value), rcl:R-EU_R0805
- C3: device rcl:C-EUC0805 -> rcl:CPOL-EUE2.5-7
- C4, C5: device rcl:CPOL-EUE2,5-6E -> rcl:CPOL-EUE2.5-7
- D1: value CGRM4001-G -> (none); device diode:CGRM4001-G -> microbuilder:DIODESOD-123
- D2: value 0805DIODE -> CGRM4001-G; device jasons_stuff:0805DIODE -> diode:CGRM4001-G
- D3: value 0805DIODE -> (none); device jasons_stuff:0805DIODE -> microbuilder:DIODESOD-123
- IC1: value PIC16F1825SO14 -> SP34063A_BOOST_REG; device jasons_stuff:PIC16F1825SO14 -> jason_eagle6:SP34063A_BOOST_REG
- IC2: value REG1117 -> PIC16F1825SO14; device burr-brown:REG1117 -> jasons_stuff:PIC16F1825SO14
- L1: device led:LED3MM -> SparkFun:INDUCTOR1210
- L2: device led:LED3MM -> inductors:DR1030
- renumbered L3 to C, L4 to D, L5 to E, L6 to F, L7 to G, L8 to H, RR7 to R7, RR8 to R8
Connections:
- removed net N$43: C2.1, C4.+, IC2.VIN, IC4.+
- new net +9V: C5.+, D1.C, IC1.VCC, R11.1
- new net N$42: D1.A, U$9.BARREL
- new net N$44: IC1.DR_C, IC1.SENS, IC1.SW_C, R11.2
- new net N$45: C1.1, IC1.TC
- new net N$57: C4.+, L1.1, L2.1, R12.1
- net BUTTON: now also IC2.RA5; no longer IC1.RA5
- net GND: now also C3.-, D2.A, IC1.GND, IC2.VSS, R13.1, R14.1, U$9.PIN; no longer C3.2, IC1.VSS, IC2.GND, IC4.-, R11.1
- net LED: now also IC2.RA4/SDO; no longer IC1.RA4/SDO
- net MIDI_IN: now also IC2.RC5/RX, R16.2; no longer IC1.RC5/RX, R12.2
- net N$10: now also D12.P$1; no longer D10.P$1
- net N$15: now also D10.P$1; no longer D8.P$1
- net N$16: now also D9.P$1; no longer D7.P$1
- net N$17: now also R22.1; no longer R19.1
- net N$18: now also R21.1; no longer R18.1
- net N$24: now also D8.P$1; no longer D6.P$1
- net N$25: now also D7.P$1; no longer D5.P$1
- net N$26: now also R20.1; no longer R17.1
- net N$27: now also R19.1; no longer R16.1
- net N$33: now also D6.P$1; no longer D4.P$1
- net N$34: now also D5.P$1; no longer D3.P$1
- net N$35: now also R18.1; no longer R15.1
- net N$36: now also R17.1; no longer R14.1
- net N$37: now also D4.P$1; no longer D2.P$1
- net N$38: now also R15.1; no longer R13.1
- net N$39: now also D4.P$2, R15.2; no longer D2.P$2, R13.2
- net N$40: now also R14.2; no longer R11.2
- net N$41: now also R1.1; no longer R3.1
- net N$46: now also D2.C, IC1.SW_E, L2.2; no longer IC4.AC1, U$9.BARREL
- net N$47: now also IC1.COMP, R12.2, R13.2; no longer IC4.AC2, U$9.PIN
- net N$48: now also R2.1; no longer R4.1
- net N$49: now also A.C; no longer L1.C
- net N$50: now also B.C; no longer L2.C
- net N$55: now also R4.1; no longer R2.1
- net N$56: now also R3.1; no longer R1.1
- net N$6: now also D11.P$1; no longer D9.P$1
- net N$7: now also R24.1; no longer R21.1
- net N$8: now also R23.1; no longer R20.1
- net SUPPLY: now also C3.+, D11.P$2, D12.P$2, D3.A, L1.2; no longer C1.1, C5.+, D1.A, D3.P$2, D4.P$2, IC2.VOUT
- net TRIG1: now also A.A, IC2.RA0/ICSPDAT, R24.2; no longer IC1.RA0/ICSPDAT, L1.A, R21.2
- net TRIG2: now also B.A, IC2.RA1/ICPCLK, R23.2; no longer IC1.RA1/ICPCLK, L2.A, R20.2
- net TRIG3: now also IC2.RC2, R22.2; no longer IC1.RC2, R19.2
- net TRIG4: now also IC2.RC1/SDA/SDI, R21.2; no longer IC1.RC1/SDA/SDI, R18.2
- net TRIG5: now also IC2.RCO/SCL/SCK, R20.2; no longer IC1.RCO/SCL/SCK, R17.2
- net TRIG6: now also IC2.RA2/INT, R19.2; no longer IC1.RA2/INT, R16.2
- net TRIG7: now also IC2.RC3/SS#, R18.2; no longer IC1.RC3/SS#, R15.2
- net TRIG8: now also IC2.RC4/TX, R17.2; no longer IC1.RC4/TX, R14.2
- net VDD: now also C2.1, D3.C, IC2.VDD, R16.1; no longer C3.1, D1.C, IC1.VDD, R12.1
- net VPP: now also IC2.RA3/MCLR#/VPP; no longer IC1.RA3/MCLR#/VPP
Other:
- note added: "POWER SUPPLY"
- moved on the sheet: C1, C2, C4, C5, D1, R1, R11, R12, R13, R14, R15, R16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
